File: BPS6001 Classic Computing Shield/BPS6001 Classic Computing Shield.brd (EAGLE design)
At the start: 119.4 x 58.7 mm, 83 parts, among them IC1 MAX3232CSE, U1 AMEGA_SHIELD_NOANALOGNO_ANALOG

Commit message: Classic Computing Shield 1.0
Parts:
- added CFG1: (no value), jumper:JP5Q
- added GROVE1: (no value), GadgetFactory_6.0:CONNECTOR_4P-LEADED-2.0
- R23, R24, R25: device GadgetFactory_6.0:0805 -> GadgetFactory_6.0:0603
- moved U$1 1.30 mm to (89.9, 52.1)
Connections:
- net 3V3: now also CFG1.10, CFG1.2, CFG1.4, CFG1.6, CFG1.8
- net 5V0: now also GROVE1.3
- net GND: now also GROVE1.4
- net JS1_5: now also GROVE1.2
- net JS1_9: now also GROVE1.1
- net RESET: now also CFG1.9
- net SW_DOWN: now also CFG1.5
- net SW_LEFT: now also CFG1.1
- net SW_RIGHT: now also CFG1.7
- net SW_UP: now also CFG1.3
Routing:
- net SW_RIGHT: track 32.6 -> 65.2 mm
- net SW_UP: track 28.2 -> 57.1 mm
- net RESET: track 19.0 -> 46.7 mm, vias 0 -> 1
- net 5V0: track 38.9 -> 60.0 mm
- net JS1_9: track 45.2 -> 61.0 mm
- net SW_LEFT: track 41.3 -> 55.8 mm
- net SW_DOWN: track 54.8 -> 68.4 mm
- net JS1_5: track 54.1 -> 56.0 mm
- net SD_CD: track 38.3 -> 40.2 mm
- net SD_MOSI: track 54.3 -> 55.8 mm
- net SD_MISO: track 51.1 -> 52.1 mm
Other:
- board text added: "6/17/2014"
- board text removed: "TODO: Mounting holes"
- board text removed: "TODO: Switches"

Commit message: Added BOM for Classic Computing Shield V1.0
Parts:
- C1, C2, C8, C9: value 4.7nF -> 4700pF
- JS1, JS2, SP1: value (none) -> Serial Port
- R23, R24, R25: value 50K -> 47K
- X1: value (none) -> VGA

Commit message: Update BOM - Classic Computing Shield.
Parts:
- H1: value AMEGA_SHIELD_NOANALOGNO_ANALOG -> Arduino Mega Header
- renumbered U1 to H1
