File: BPS6001 Classic Computing Shield/BPS6001 Classic Computing Shield.sch (EAGLE design)
At the start: 80 parts, among them IC1 MAX3232CSE, U1 AMEGA_SHIELD_NOANALOGNO_ANALOG

Commit message: Classic Computing Shield 1.0
Parts:
- added CFG1: (no value), jumper:JP5Q
- added GROVE1: (no value), GadgetFactory_6.0:CONNECTOR_TWIG-2.0-LEADED
- R23, R24, R25: device GadgetFactory_6.0:R0805 -> GadgetFactory_6.0:R0603
Connections:
- net 3V3: now also CFG1.10, CFG1.2, CFG1.4, CFG1.6, CFG1.8
- net 5V0: now also GROVE1.3
- net GND: now also GROVE1.4
- net JS1_5: now also GROVE1.2
- net JS1_9: now also GROVE1.1
- net RESET: now also CFG1.9
- net SW_DOWN: now also CFG1.5
- net SW_LEFT: now also CFG1.1
- net SW_RIGHT: now also CFG1.7
- net SW_UP: now also CFG1.3
Other:
- note added: "Seeed Grove Connector"
- note removed: "TODO: Add Jumpers to buttons TODO: Put buttons on Joystick pins? TODO: Add Grove Connector TODO: Change silkscreen of the buttons TODO: Consider adding thumb joystick"
Changed lines of the file:
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@@
 <part name="3V3_PWR9" library="GadgetFactory_all" deviceset="3V3" device=""/>
 <part name="FRAME2" library="frames" deviceset="A3L-LOC" device=""/>
-<part name="R23" library="GadgetFactory_6.0" deviceset="R" device="0805" value="50K"/>
-<part name="R24" library="GadgetFactory_6.0" deviceset="R" device="0805" value="50K"/>
-<part name="R25" library="GadgetFactory_6.0" deviceset="R" device="0805" value="50K"/>
+<part name="R23" library="GadgetFactory_6.0" deviceset="R" device="0603" value="50K"/>
+<part name="R24" library="GadgetFactory_6.0" deviceset="R" device="0603" value="50K"/>
+<part name="R25" library="GadgetFactory_6.0" deviceset="R" device="0603" value="50K"/>
 <part name="3V3_PWR10" library="GadgetFactory_all" deviceset="3V3" device=""/>
 <part name="FRAME3" library="frames" deviceset="A3L-LOC" device=""/>
@@
 <part name="R47" library="GadgetFactory_6.0" deviceset="R" device="0603" value="390"/>
 <part name="R48" library="GadgetFactory_6.0" deviceset="R" device="0603" value="390"/>
+<part name="GROVE1" library="GadgetFactory_6.0" deviceset="CONNECTOR_TWIG-2.0-LEADED" device=""/>
+<part name="CFG1" library="jumper" deviceset="JP5Q" device=""/>
+<part name="3V3_PWR7" library="GadgetFactory_all" deviceset="3V3" device=""/>
 </parts>
 <sheets>
@@
 <text x="297.18" y="30.48" size="2.1844" layer="91">Copyright 2010-2011 Gadget Factory, LLC</text>
 <text x="290.83" y="26.67" size="1.778" layer="91">See more details at www.GadgetFactory.net</text>
-<text x="177.8" y="228.6" size="1.778" layer="91">TODO: Add Jumpers to buttons
-TODO: Put buttons on Joystick pins?
-TODO: Add Grove Connector
-TODO: Change silkscreen of the buttons
-TODO: Consider adding thumb joystick</text>
+<text x="172.72" y="68.58" size="1.778" layer="91">Seeed Grove Connector</text>
 </plain>
 <instances>
@@
 <instance part="R47" gate="A" x="33.02" y="93.98"/>
 <instance part="R48" gate="A" x="33.02" y="83.82"/>
+<instance part="GROVE1" gate="G$1" x="198.12" y="58.42"/>
+<instance part="CFG1" gate="B" x="68.58" y="162.56"/>
+<instance part="3V3_PWR7" gate="A" x="68.58" y="175.26"/>
 </instances>
 <busses>
@@
 <wire x1="177.8" y1="96.52" x2="182.88" y2="96.52" width="0.1524" layer="91"/>
 </segment>
+<segment>
+<pinref part="GROVE1" gate="G$1" pin="4"/>
+<wire x1="194.31" y1="54.61" x2="189.23" y2="54.61" width="0.2032" layer="91"/>
+<label x="189.23" y="54.61" size="1.778" layer="95"/>
+</segment>
 </net>
 <net name="BLUE2" class="0">
@@
 <segment>
 <wire x1="43.18" y1="119.38" x2="40.64" y2="119.38" width="0.1524" layer="91"/>
-<wire x1="40.64" y1="119.38" x2="38.1" y2="119.38" width="0.1524" layer="91"/>
 <pinref part="S3" gate="G$1" pin="P1"/>
 <pinref part="R9" gate="A" pin="2"/>
 <pinref part="S3" gate="G$1" pin="P"/>
+<pinref part="CFG1" gate="B" pin="1"/>
+<wire x1="63.5" y1="154.94" x2="33.02" y2="154.94" width="0.1524" layer="91"/>
+<wire x1="33.02" y1="154.94" x2="33.02" y2="119.38" width="0.1524" layer="91"/>
+<wire x1="33.02" y1="119.38" x2="40.64" y2="119.38" width="0.1524" layer="91"/>
 </segment>
 <segment>
@@
 <segment>
 <wire x1="55.88" y1="119.38" x2="53.34" y2="119.38" width="0.1524" layer="91"/>
-<wire x1="53.34" y1="119.38" x2="50.8" y2="119.38" width="0.1524" layer="91"/>
 <pinref part="S1" gate="G$1" pin="P1"/>
 <pinref part="R10" gate="A" pin="2"/>
 <pinref part="S1" gate="G$1" pin="P"/>
+<pinref part="CFG1" gate="B" pin="3"/>
+<wire x1="66.04" y1="154.94" x2="66.04" y2="152.4" width="0.1524" layer="91"/>
+<wire x1="66.04" y1="152.4" x2="48.26" y2="152.4" width="0.1524" layer="91"/>
+<wire x1="48.26" y1="152.4" x2="48.26" y2="119.38" width="0.1524" layer="91"/>
+<wire x1="48.26" y1="119.38" x2="53.34" y2="119.38" width="0.1524" layer="91"/>
 </segment>
 <segment>
@@
 <segment>
 <wire x1="69.85" y1="119.38" x2="67.31" y2="119.38" width="0.1524" layer="91"/>
-<wire x1="67.31" y1="119.38" x2="64.77" y2="119.38" width="0.1524" layer="91"/>
+<wire x1="67.31" y1="119.38" x2="66.04" y2="119.38" width="0.1524" layer="91"/>
 <pinref part="S4" gate="G$1" pin="P1"/>
 <pinref part="R17" gate="A" pin="2"/>
 <pinref part="S4" gate="G$1" pin="P"/>
+<pinref part="CFG1" gate="B" pin="5"/>
+<wire x1="66.04" y1="119.38" x2="64.77" y2="119.38" width="0.1524" layer="91"/>
+<wire x1="68.58" y1="154.94" x2="68.58" y2="149.86" width="0.1524" layer="91"/>
+<wire x1="68.58" y1="149.86" x2="60.96" y2="149.86" width="0.1524" layer="91"/>
+<wire x1="60.96" y1="149.86" x2="60.96" y2="119.38" width="0.1524" layer="91"/>
+<wire x1="60.96" y1="119.38" x2="64.77" y2="119.38" width="0.1524" layer="91"/>
 </segment>
 <segment>
@@
 <segment>
 <wire x1="97.79" y1="119.38" x2="95.25" y2="119.38" width="0.1524" layer="91"/>
-<wire x1="95.25" y1="119.38" x2="92.71" y2="119.38" width="0.1524" layer="91"/>
+<wire x1="95.25" y1="119.38" x2="93.98" y2="119.38" width="0.1524" layer="91"/>
 <pinref part="S2" gate="G$1" pin="P1"/>
 <pinref part="R11" gate="A" pin="2"/>
 <pinref part="S2" gate="G$1" pin="P"/>
+<pinref part="CFG1" gate="B" pin="9"/>
+<wire x1="93.98" y1="119.38" x2="92.71" y2="119.38" width="0.1524" layer="91"/>
+<wire x1="73.66" y1="154.94" x2="88.9" y2="154.94" width="0.1524" layer="91"/>
+<wire x1="88.9" y1="154.94" x2="88.9" y2="119.38" width="0.1524" layer="91"/>
+<wire x1="88.9" y1="119.38" x2="92.71" y2="119.38" width="0.1524" layer="91"/>
 </segment>
 <segment>
@@
 <pinref part="3V3_PWR6" gate="A" pin="3V3"/>
 </segment>
+<segment>
+<pinref part="CFG1" gate="B" pin="2"/>
+<pinref part="CFG1" gate="B" pin="4"/>
+<wire x1="63.5" y1="170.18" x2="66.04" y2="170.18" width="0.1524" layer="91"/>
+<pinref part="CFG1" gate="B" pin="6"/>
+<wire x1="66.04" y1="170.18" x2="68.58" y2="170.18" width="0.1524" layer="91"/>
+<pinref part="CFG1" gate="B" pin="8"/>
+<wire x1="68.58" y1="170.18" x2="71.12" y2="170.18" width="0.1524" layer="91"/>
+<pinref part="CFG1" gate="B" pin="10"/>
+<wire x1="71.12" y1="170.18" x2="73.66" y2="170.18" width="0.1524" layer="91"/>
+<pinref part="3V3_PWR7" gate="A" pin="3V3"/>
+<wire x1="73.66" y1="170.18" x2="68.58" y2="170.18" width="0.1524" layer="91"/>
+<wire x1="68.58" y1="170.18" x2="68.58" y2="172.72" width="0.1524" layer="91"/>
+</segment>
 </net>
 <net name="JS1_6" class="0">
@@
 <pinref part="5V0_PWR1" gate="A" pin="5V0"/>
 </segment>
+<segment>
+<pinref part="GROVE1" gate="G$1" pin="3"/>
+<wire x1="194.31" y1="57.15" x2="189.23" y2="57.15" width="0.2032" layer="91"/>
+<label x="189.23" y="57.15" size="1.778" layer="95"/>
+</segment>
 </net>
 <net name="SD_CD" class="0">
@@
 <pinref part="U1" gate="G$1" pin="D7"/>
 </segment>
+<segment>
+<pinref part="GROVE1" gate="G$1" pin="1"/>
+<wire x1="194.31" y1="62.23" x2="176.276" y2="62.23" width="0.2032" layer="91"/>
+<label x="177.8" y="63.5" size="1.778" layer="95"/>
+</segment>
 </net>
 <net name="JS1_5" class="0">
@@
 <label x="180.34" y="160.02" size="1.778" layer="95" rot="R90"/>
 <pinref part="U1" gate="G$1" pin="D6"/>
+</segment>
+<segment>
+<pinref part="GROVE1" gate="G$1" pin="2"/>
+<wire x1="194.31" y1="59.69" x2="176.276" y2="59.69" width="0.2032" layer="91"/>
+<label x="177.8" y="60.198" size="1.778" layer="95"/>
 </segment>
 </net>
@@
 <segment>
 <wire x1="82.55" y1="119.38" x2="80.01" y2="119.38" width="0.1524" layer="91"/>
-<wire x1="80.01" y1="119.38" x2="77.47" y2="119.38" width="0.1524" layer="91"/>
+<wire x1="80.01" y1="119.38" x2="78.74" y2="119.38" width="0.1524" layer="91"/>
 <pinref part="S5" gate="G$1" pin="P1"/>
 <pinref part="R18" gate="A" pin="2"/>
 <pinref part="S5" gate="G$1" pin="P"/>
+<pinref part="CFG1" gate="B" pin="7"/>
+<wire x1="78.74" y1="119.38" x2="77.47" y2="119.38" width="0.1524" layer="91"/>
+<wire x1="71.12" y1="154.94" x2="71.12" y2="147.32" width="0.1524" layer="91"/>
+<wire x1="71.12" y1="147.32" x2="73.66" y2="147.32" width="0.1524" layer="91"/>
+<wire x1="73.66" y1="147.32" x2="73.66" y2="119.38" width="0.1524" layer="91"/>
+<wire x1="73.66" y1="119.38" x2="77.47" y2="119.38" width="0.1524" layer="91"/>
 </segment>
 </net>
@@
 </nets>
 </sheet>
+<sheet>
+<plain>
+</plain>
+<instances>
+</instances>
+<busses>
+</busses>
+<nets>
+</nets>
+</sheet>

Commit message: Added BOM for Classic Computing Shield V1.0
Parts:
- AJ1, AJ2: PARTNO (none) -> 3440030P1
- C1, C2, C8, C9: value 4.7nF -> 4700pF; PARTNO (none) -> C0603C472J5RACTU
- C3, C4, C5, C6, C7: PARTNO (none) -> GRM21BR71E104KA01L
- CFG1: PARTNO (none) -> M20-9720545
- GROVE1: PARTNO (none) -> ACC39145O
- IC1: PARTNO (none) -> MAX3232ECDR
- JS1, JS2, SP1: value (none) -> Serial Port; PARTNO (none) -> 10090097-P094VLF
- LED1, LED2, LED3, LED4: PARTNO (none) -> LTST-C190GKT
- LOGO1, PWR_1, PWR_2, U1: BOM (none) -> EXCLUDE
- PS2_A, PS2_B: PARTNO (none) -> MD-60S
- R1, R10, R11, R12, R13, R14, R15, R16, R17, R18, R19, R2, R20, R21, R3, R4, R5, R6, R7, R8, R9: PARTNO (none) -> RMCF0603JT47K0
- R22, R28, R45, R46: PARTNO (none) -> RMCF0603JT3K30
- R23, R24, R25: value 50K -> 47K; PARTNO (none) -> RMCF0603JT47K0
- R26, R27, R43, R44, R47, R48: PARTNO (none) -> RMCF0603JT390R
- R29, R30: PARTNO (none) -> RMCF0603FT82R5
- R31, R35, R42: PARTNO (none) -> RMCF0603JT3K90
- R32, R36, R41: PARTNO (none) -> RMCF0603JT2K00
- R33, R37, R40: PARTNO (none) -> RMCF0603JT1K00
- R34, R38, R39: PARTNO (none) -> RMCF0603JT510R
- S1, S2, S3, S4, S5: PARTNO (none) -> PTS525SM10SMTR LFS
- SD1: PARTNO (none) -> 101-00660-68-6
- X1: value (none) -> VGA; PARTNO (none) -> 1-1734530-1

Commit message: Update BOM - Classic Computing Shield.
Parts:
- H1: value AMEGA_SHIELD_NOANALOGNO_ANALOG -> Arduino Mega Header; BOM EXCLUDE -> (none); PARTNO (none) -> Arduino_Mega_Header
- renumbered U1 to H1

Commit message: Fix the PS/2 connectors.
Parts:
- PS2_A, PS2_B: value CON_PS/2 -> MINI-DIN6PTH; device usb1:CON_PS/2 -> SparkFun-Connectors:MINI-DIN6PTH; PARTNO MD-60S -> (none)
Connections:
- net 5V0: now also PS2_A.4; no longer PS2_A.VCC
- net 5V0_PS2: now also PS2_B.4; no longer PS2_B.VCC
- net GND: now also PS2_A.3; no longer PS2_A.GND
- net JOY_GND: now also PS2_B.3; no longer PS2_B.GND
- net N$16: now also PS2_B.1; no longer PS2_B.DATA
- net N$17: now also PS2_B.5; no longer PS2_B.CLK
- net PS2CLK1: now also PS2_A.5; no longer PS2_A.CLK
- net PS2DAT1: now also PS2_A.1; no longer PS2_A.DATA
Changed lines of the file:
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@@
 <attribute name="BOM" value="EXCLUDE"/>
-</part>
-<part name="PS2_B" library="usb1" deviceset="CON_PS/2" device="">
-<attribute name="PARTNO" value="MD-60S"/>
-</part>
-<part name="PS2_A" library="usb1" deviceset="CON_PS/2" device="">
-<attribute name="PARTNO" value="MD-60S"/>
 </part>
 <part name="R9" library="GadgetFactory" deviceset="R" device="0603" value="47K">
@@
 </part>
 <part name="3V3_PWR7" library="GadgetFactory_all" deviceset="3V3" device=""/>
+<part name="PS2_B" library="SparkFun-Connectors" deviceset="MINI-DIN6" device="PTH"/>
+<part name="PS2_A" library="SparkFun-Connectors" deviceset="MINI-DIN6" device="PTH"/>
 </parts>
 <sheets>
@@
 <instance part="LOGO1" gate="G$1" x="292.1" y="30.48">
 <attribute name="BOM" x="292.1" y="30.48" size="1.778" layer="96" display="off"/>
-</instance>
-<instance part="PS2_B" gate="1" x="48.26" y="88.9">
-<attribute name="PARTNO" x="48.26" y="88.9" size="1.778" layer="96" display="off"/>
-</instance>
-<instance part="PS2_A" gate="1" x="104.14" y="88.9">
-<attribute name="PARTNO" x="104.14" y="88.9" size="1.778" layer="96" display="off"/>
 </instance>
 <instance part="R9" gate="A" x="43.18" y="114.3" smashed="yes" rot="R90">
@@
 </instance>
 <instance part="3V3_PWR7" gate="A" x="68.58" y="175.26"/>
+<instance part="PS2_B" gate="G$1" x="45.72" y="88.9" rot="R180"/>
+<instance part="PS2_A" gate="G$1" x="99.06" y="88.9" rot="R180"/>
 </instances>
 <busses>
@@
 </segment>
 <segment>
-<pinref part="PS2_A" gate="1" pin="GND"/>
 <pinref part="GND19" gate="A" pin="GND"/>
+<pinref part="PS2_A" gate="G$1" pin="3"/>
+<junction x="93.98" y="88.9"/>
+<pinref part="PS2_A" gate="G$1" pin="3"/>
 </segment>
 <segment>
@@
 <wire x1="83.82" y1="93.98" x2="93.98" y2="93.98" width="0.2032" layer="91"/>
 <label x="69.85" y="93.98" size="1.778" layer="95"/>
-<pinref part="PS2_A" gate="1" pin="DATA"/>
+<pinref part="PS2_A" gate="G$1" pin="1"/>
 </segment>
 <segment>
@@
 <wire x1="83.82" y1="83.82" x2="93.98" y2="83.82" width="0.2032" layer="91"/>
 <label x="69.85" y="83.82" size="1.778" layer="95"/>
-<pinref part="PS2_A" gate="1" pin="CLK"/>
+<pinref part="PS2_A" gate="G$1" pin="5"/>
 </segment>
 <segment>
@@
 <net name="5V0" class="0">
 <segment>
-<pinref part="PS2_A" gate="1" pin="VCC"/>
 <pinref part="5V0_PWR10" gate="A" pin="5V0"/>
+<pinref part="PS2_A" gate="G$1" pin="4"/>
+<junction x="93.98" y="86.36"/>
+<pinref part="PS2_A" gate="G$1" pin="4"/>
 </segment>
 <segment>
@@
 </segment>
 <segment>
-<pinref part="PS2_B" gate="1" pin="GND"/>
 <pinref part="GND18" gate="A" pin="GND"/>
-<wire x1="35.56" y1="88.9" x2="38.1" y2="88.9" width="0.1524" layer="91"/>
+<wire x1="35.56" y1="88.9" x2="40.64" y2="88.9" width="0.1524" layer="91"/>
+<pinref part="PS2_B" gate="G$1" pin="3"/>
 </segment>
 <segment>
@@
 <net name="5V0_PS2" class="0">
 <segment>
-<pinref part="PS2_B" gate="1" pin="VCC"/>
 <pinref part="5V0_PWR9" gate="A" pin="5V0"/>
-<wire x1="33.02" y1="86.36" x2="38.1" y2="86.36" width="0.1524" layer="91"/>
+<wire x1="33.02" y1="86.36" x2="40.64" y2="86.36" width="0.1524" layer="91"/>
+<pinref part="PS2_B" gate="G$1" pin="4"/>
 </segment>
 <segment>
@@
 <net name="N$16" class="0">
 <segment>
-<pinref part="PS2_B" gate="1" pin="DATA"/>
 <pinref part="R47" gate="A" pin="2"/>
+<pinref part="PS2_B" gate="G$1" pin="1"/>
+<wire x1="40.64" y1="93.98" x2="38.1" y2="93.98" width="0.1524" layer="91"/>
 </segment>
 </net>
 <net name="N$17" class="0">
 <segment>
-<pinref part="PS2_B" gate="1" pin="CLK"/>
 <pinref part="R48" gate="A" pin="2"/>
-</segment>
-</net>
+<pinref part="PS2_B" gate="G$1" pin="5"/>
+<wire x1="40.64" y1="83.82" x2="38.1" y2="83.82" width="0.1524" layer="91"/>
+</segment>
+</net>
