File: BPM7001 Arcade MegaWing/BPW5031 Arcade MegaWing.sch (EAGLE design)
At the start: 61 parts, among them SW1 TPA-5POS

Commit message: Arcade MegaWing V1.3
Parts:
- removed AH, AL: WING8WING8_NOHOLES, Papilio:WING8WING8_NOHOLES
- removed AUDIO1: AUDIOJACK, GadgetFactory:AUDIOJACK
- removed SW1: TPA-5POS, GadgetFactory:TPA-5POS
- removed U$3, U$4: MINI-DIN6PTH, SparkFun-Connectors:MINI-DIN6PTH
- added AUDIO: AUDIOJACK, GadgetFactory_6.0:AUDIOJACK
- added J1: COCOON_48BIT_WINGSIDE, usb1:COCOON_48BIT_WINGSIDE
- added LED1, LED2, LED3, LED4: (no value), led:LEDCHIPLED_0603
- added R45: 390, GadgetFactory:R0603
- added S4, S5: (no value), opto:10-XX
- R1: value 390 -> 3.9K
- R10: value 3.9K -> 510
- R11: value 2K -> 1K
- R12: value 1K -> 510
- R13: value 510 -> 1K
- R14: value 47K -> 510
- R15: value 47K -> 3.3K
- R16: value 3.9K -> 3.3K
- R17, R21: value 2K -> 390
- R18, R22: value 1K -> 390
- R19, R23: value 510 -> 390
- R2, R3: value 3.3K -> 3.9K
- R20: value 3.9K -> 390
- R24, R26, R27, R29, R30, R31, R32, R37, R38, R39, R40, R42, R43, R44: value 47K -> 390
- R25, R28: value 82.5 -> 390
- R4, R5: value 390 -> 82.5
- R6: value 390 -> 2K
- R7, R8: value 47K -> 2K
- R9: value 47K -> 1K
- U$1: value MEGAWING_HALF_P1 -> MINI-DIN6PTH; device Papilio:MEGAWING_HALF_P1 -> SparkFun-Connectors:MINI-DIN6PTH
- U$2: value MICROSD -> MINI-DIN6PTH; device adafruit:MICROSD -> SparkFun-Connectors:MINI-DIN6PTH
- X1: device GadgetFactory:F15HDH -> GadgetFactory_6.0:F15HDH
- renumbered LOGO1 to LOGO2
Connections:
- removed net BLUE0: R20A.1, U$1B_IO.A3
- removed net GREEN0: R16A.1, U$1B_IO.A7
- removed net JOY_3V3: AH.3V3, AL.3V3, R29A.2, R30A.2, R31A.2, R32A.2, R33A.2, R34A.2, R35A.2, R36A.2, R37A.2, R38A.2, R39A.2, R40A.2, R41A.2, R42A.2, R43A.2, R44A.2
- removed net JOY_DOWN: R24A.2, SW1.DOWN, U$1B_IO.A16
- removed net JOY_FIRE1: R8A.2, S1.P, S1.P1, U$1C_IO.A12
- removed net JOY_FIRE2: R9A.2, S3.P, S3.P1, U$1B_IO.A11
- removed net JOY_GND: AH.GND, AL.GND, JS1.8, JS2.8
- removed net JOY_LEFT: R14A.2, SW1.LEFT, U$1B_IO.A12
- removed net JOY_RIGHT: R15A.2, SW1.RIGHT, U$1B_IO.A13
- removed net JOY_SEL: R27A.2, SW1.SELECT, U$1B_IO.A14
- removed net JOY_UP: R26A.2, SW1.UP, U$1B_IO.A15
- removed net N$2: AH.5, JS1.2, R32A.1
- removed net N$24: AH.1, JS1.9, R36A.1
- removed net N$7: AH.8, JS1.5, R29A.1
- removed net N$8: AH.3, JS1.6, R34A.1
- removed net RED0: R10A.1, U$1C_IO.A7
- removed net SD_!CS: U$1C_IO.A13, U$2.CS
- removed net SD_DI: U$1C_IO.A14, U$2.DATA_IN
- removed net SD_DO: U$1C_IO.A16, U$2.DATA_OUT
- removed net SD_SCK: U$1C_IO.A15, U$2.SCLK
- new net BLUE4: J1WING1.B4, R14A.1
- new net GREEN4: J1WING1.B8, R12A.1
- new net JS1_1: J1WING1.B13, R32A.1
- new net JS1_2: J1WING1.B15, R31A.1
- new net JS1_3: J1WING1.B16, R30A.1
- new net JS1_4: J1WING1.A2, R29A.1
- new net JS1_5: J1WING1.A4, R28A.1
- new net JS1_6: J1WING1.B14, R27A.1
- new net JS1_8: J1WING1.A1, R26A.1
- new net JS1_9: J1WING1.A3, R25A.1
- new net JS2_1: J1WING2.A9, R24A.1
- new net JS2_2: J1WING2.A11, R23A.1
- new net JS2_3: J1WING2.A12, R22A.1
- new net JS2_4: J1WING2.A14, R21A.1
- new net JS2_5: J1WING2.A16, R20A.1
- new net JS2_6: J1WING2.A10, R19A.1
- new net JS2_8: J1WING2.A13, R18A.1
- new net JS2_9: J1WING2.A15, R17A.1
- new net LED1: J1WING1.A8, R37A.2
- new net LED2: J1WING1.A7, R38A.2
- new net LED3: J1WING1.A6, R39A.2
- new net LED4: J1WING1.A5, R40A.2
- new net N$32: JS1.1, R24A.2
- new net N$33: JS1.2, R23A.2
- new net N$34: JS1.3, R22A.2
- new net N$35: JS1.4, R21A.2
- new net N$36: JS1.5, R20A.2
- new net N$37: JS1.9, R17A.2
- new net N$38: JS1.6, R19A.2
- new net N$39: JS1.8, R18A.2
- new net RED4: J1WING2.A8, R10A.1
- new net SW1: J1WING1.B9, R33A.2, S1.P, S1.P1
- new net SW2: J1WING1.B10, R34A.2, S2.P, S2.P1
- new net SW3: J1WING1.B11, R35A.2, S3.P, S3.P1
- new net SW4: J1WING1.B12, R36A.2, S4.P, S4.P1
- net 3V3: now also J1G$1.3V3, J1G$2.3V3, J1G$3.3V3, J1G$4.3V3, J1G$5.3V3, J1G$6.3V3, S4.S1, S5.S1; no longer R14A.1, R15A.1, R24A.1, R26A.1, R27A.1, U$1B_POWER.3V3@P3, U$1B_POWER.3V3@P7, U$1C_POWER.3V3@P3, U$1C_POWER.3V3@P7, U$2.VDD
- net 5V0: now also J1G$1.5V, J1G$2.5V, J1G$3.5V, J1G$4.5V, J1G$5.5V, J1G$6.5V, JS1.7, JS2.7, U$1.4, U$2.4; no longer U$1C_POWER.5V0@P4, U$3.4, U$4.4
- net AUDIO+: now also J1WING1.A15, R16A.2; no longer R3A.2, U$1C_IO.A1
- net AUDIO-: now also J1WING1.A16, R15A.2; no longer R2A.2, U$1C_IO.A2
- net BLUE: now also R13A.2, R14A.2, R3A.2, R8A.2; no longer R20A.2, R21A.2, R22A.2, R23A.2
- net BLUE1: now also J1WING1.B1, R3A.1; no longer R21A.1, U$1B_IO.A4
- net BLUE2: now also J1WING1.B2, R8A.1; no longer R22A.1, U$1B_IO.A5
- net BLUE3: now also J1WING1.B3, R13A.1; no longer R23A.1, U$1B_IO.A6
- net GND: now also AUDIO.1, J1G$1.GND, J1G$2.GND, J1G$3.GND, J1G$4.GND, J1G$5.GND, J1G$6.GND, LED1.C, LED2.C, LED3.C, LED4.C, R33A.1, R34A.1, R35A.1, R36A.1, R41A.1, U$1.3, U$2.3; no longer AUDIO1.1, R7A.1, R8A.1, R9A.1, SW1.COM1, SW1.COM2, U$1B_POWER.GND@P1, U$1B_POWER.GND@P5, U$1C_POWER.GND@P1, U$1C_POWER.GND@P5, U$2.GND, U$2.GND1, U$2.VSS, U$3.3, U$4.3
- net GREEN: now also R11A.2, R12A.2, R2A.2, R7A.2; no longer R16A.2, R17A.2, R18A.2, R19A.2
- net GREEN1: now also J1WING1.B5, R2A.1; no longer R17A.1, U$1B_IO.A8
- net GREEN2: now also J1WING1.B6, R7A.1; no longer R18A.1, U$1B_IO.A9
- net GREEN3: now also J1WING1.B7, R11A.1; no longer R19A.1, U$1B_IO.A10
- net HORIZONTAL_SYNC: now also J1WING2.A4, R4A.1; no longer R28A.1, U$1B_IO.A1
- net N$1: now also AUDIO.3, C2.1, R15A.1; no longer AH.4, JS1.1, R33A.1
- net N$10: now also LED3.A, R39A.1; no longer AUDIO1.2, C2.1, R3A.1
- net N$11: now also LED4.A, R40A.1; no longer AUDIO1.3, C1.1, R2A.1
- net N$12: now also R42A.2, U$2.1; no longer R6A.2, U$3.1
- net N$13: now also R43A.2, U$2.5; no longer R5A.2, U$3.5
- net N$14: now also R44A.2, U$1.1; no longer R4A.2, U$4.1
- net N$15: now also R45A.2, U$1.5; no longer R1A.2, U$4.5
- net N$16: now also R32A.2; no longer AL.4, R41A.1
- net N$17: now also R31A.2; no longer AL.5, R40A.1
- net N$18: now also R30A.2; no longer AL.6, R39A.1
- net N$19: now also R29A.2; no longer AL.7, R38A.1
- net N$20: now also R28A.2; no longer AL.8, R37A.1
- net N$21: now also JS2.9, R25A.2; no longer AL.3, JS2.6, R42A.1
- net N$22: now also JS2.6, R27A.2; no longer AL.2, JS2.7, R43A.1
- net N$23: now also JS2.8, R26A.2; no longer AL.1, JS2.9, R44A.1
- net N$3: now also LED1.A, R37A.1; no longer AH.6, JS1.3, R31A.1
- net N$4: now also R4A.2; no longer R28A.2
- net N$5: now also R5A.2; no longer R25A.2
- net N$6: now also AUDIO.2, C1.1, R16A.1; no longer AH.7, JS1.4, R30A.1
- net N$9: now also LED2.A, R38A.1; no longer AH.2, JS1.7, R35A.1
- net PS2CLK1: now also J1WING1.A14, R43A.1; no longer R5A.1, U$1C_IO.A5
- net PS2CLK2: now also J1WING2.A2, R45A.1; no longer R1A.1, U$1C_IO.A3
- net PS2DAT1: now also J1WING1.A13, R42A.1; no longer R6A.1, U$1C_IO.A6
- net PS2DAT2: now also J1WING2.A1, R44A.1; no longer R4A.1, U$1C_IO.A4
- net RED: now also R1A.2, R6A.2, R9A.2; no longer R11A.2, R12A.2, R13A.2
- net RED1: now also J1WING2.A5, R1A.1; no longer R11A.1, U$1C_IO.A8
- net RED2: now also J1WING2.A6, R6A.1; no longer R12A.1, U$1C_IO.A9
- net RED3: now also J1WING2.A7, R9A.1; no longer R13A.1, U$1C_IO.A10
- net RESET: now also J1WING1.A12, R41A.2, S5.P, S5.P1; no longer R7A.2, S2.P, S2.P1, U$1C_IO.A11
- net VERTICAL_SYNC: now also J1WING2.A3, R5A.1; no longer R25A.1, U$1B_IO.A2
Other:
- note added: "Copyright 2010-2011 Gadget Factory, LLC"
- note added: "This work is licensed under the Creative Commons Non-Commercial Attribution License."
- note removed: "Copyright 2010-2012 Gadget Factory, LLC"
- note removed: "This work is licensed under the Creative Commons Non-Commercial Attribution Share-Alike License."
- moved on the sheet: C1, C2, JS1, JS2, R24, R26, R27, R29, R30, R31, R32, S1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
